Commit message: my Commit

File: catkin_ws/src/my_robot/urdf/my_robot.xacro (robot description, xacro)
@@ -1,4 +1,4 @@
 <robot name="my_robot" xmlns:xacro="http://www.ros.org/wiki/xacro">
-  <xacro:include filename="$(find my_robot)/urdf/my_robot_Differential.gazebo" />
+  <xacro:include filename="$(find my_robot)/urdf/my_robot.gazebo" />
   <link name="robot_footprint"></link>
   <joint name="robot_footprint_joint" type="fixed">
@@ -21,5 +21,5 @@
       <origin xyz="0 0 0" rpy=" 0 0 0"/>
       <geometry>
-        <box size=".4 .2 .1"/>
+        <box size=".5 .2 .1"/>
       </geometry>
     </collision>
@@ -27,5 +27,5 @@
       <origin xyz="0 0 0" rpy=" 0 0 0"/>
       <geometry>
-        <box size=".4 .2 .1"/>
+        <box size=".5 .2 .1"/>
       </geometry>
     </visual>
@@ -56,5 +56,5 @@
   </link>
   <joint type="continuous" name="left_wheel_hinge">
-    <origin xyz="0.0 0.15 0" rpy="0 0 0"/>
+    <origin xyz="0.15 0.2 0" rpy="0 0 0"/>
     <child link="left_wheel"/>
     <parent link="chassis"/>
@@ -81,4 +81,36 @@
     </collision>
     <visual name='left_wheel_visual'>
+      <origin xyz="0 0 0" rpy=" 0 1.57079633 1.57079633"/>
+      <geometry>
+        <cylinder radius="0.1" length="0.05"/>
+      </geometry>
+    </visual>
+  </link>
+  <!-- Left Rear Dummy wheel-->
+  <joint type="continuous" name="left_rear_wheel_hinge">
+    <origin xyz="-0.15 0.2 0" rpy="0 0 0"/>
+    <child link="left_rear_wheel"/>
+    <parent link="chassis"/>
+    <axis xyz="0 1 0" rpy="0 0 0"/>
+    <limit effort="10000" velocity="1000"/>
+    <dynamics damping="1.0" friction="1.0"/>
+  </joint>
+  <link name="left_rear_wheel">
+    <inertial>
+      <mass value="5.0"/>
+      <origin xyz="0 0 0" rpy=" 0 1.57079633 1.57079633"/>
+      <inertia
+          ixx="0.1" ixy="0" ixz="0"
+          iyy="0.1" iyz="0"
+          izz="0.1"
+      />
+    </inertial>
+    <collision name='left_rear_wheel_collision'>
+      <origin xyz="0 0 0" rpy=" 0 1.57079633 1.57079633"/>
+      <geometry>
+        <cylinder radius="0.1" length="0.05"/>
+      </geometry>
+    </collision>
+    <visual name='left_rear_wheel_visual'>
       <origin xyz="0 0 0" rpy=" 0 1.57079633 1.57079633"/>
       <geometry>
@@ -91,5 +123,5 @@
     <parent link="chassis"/>
     <child link="right_wheel"/>
-    <origin xyz="0.0 -0.15 0.0" rpy="0 0 0"/>
+    <origin xyz="0.15 -0.2 0" rpy="0 0 0"/>
     <axis xyz="0 1 0"/>
     <limit effort="10000" velocity="1000"/>
@@ -113,4 +145,36 @@
     </collision>
     <visual name="right_wheel_visual">
+      <origin xyz="0 0 0" rpy="0 1.57079633 1.57079633"/>
+      <geometry>
+        <cylinder radius="0.1" length="0.05"/>
+      </geometry>
+    </visual>
+  </link>
+   <!-- Rear Dummy RIGHT WHEEL -->
+  <joint name="right_rear_wheel_hinge" type="continuous">
+    <parent link="chassis"/>
+    <child link="right_rear_wheel"/>
+    <origin xyz="-0.15 -0.2 0" rpy="0 0 0"/>
+    <axis xyz="0 1 0"/>
+    <limit effort="10000" velocity="1000"/>
+    <dynamics damping="1.0" friction="1.0"/>
+  </joint>
+  <link name="right_rear_wheel">
+    <inertial>
+      <mass value="5.0"/>
+      <origin xyz="0 0 0" rpy="0 1.57079633 1.57079633"/>
+      <inertia
+          ixx="0.1" ixy="0" ixz="0"
+          iyy="0.1" iyz="0"
+          izz="0.1"
+      />
+    </inertial>
+    <collision name="right_rear_wheel_collision">
+      <origin xyz="0 0 0" rpy="0 1.57079633 1.57079633"/>
+      <geometry>
+        <cylinder radius="0.1" length="0.05"/>
+      </geometry>
+    </collision>
+    <visual name="right_rear_wheel_visual">
       <origin xyz="0 0 0" rpy="0 1.57079633 1.57079633"/>
       <geometry>
@@ -142,9 +206,17 @@
   </link>
   <joint name="camera_joint" type="fixed">
-    <origin xyz="0.20 0 0" rpy="0 0 0" />
+    <origin xyz="0.25 0 0" rpy="0 0 0" />
     <axis xyz="0 1 0" rpy="0 0 0"/>
     <parent link="chassis"/>
     <child link="camera" />
     <imageTopicName>rgb/image_raw</imageTopicName>
+  </joint>
+  <!-- RGBD Camera -->
+  <link name="camera_link_optical">
+  </link>
+  <joint name="camera+optical_joint" type="fixed">
+    <origin xyz="0 0 0" rpy="-1.57079633 0 -1.57079633"/>
+    <parent link="camera"/>
+    <child link="camera_link_optical"/>
   </joint>
   <!--\template for LIDAR structure-->
@@ -171,5 +243,5 @@
   </link>
   <joint name="hokuyo_joint" type="fixed">
-    <origin xyz="0.15 0 0.1" rpy="0 0 0" />
+    <origin xyz="0.2 0 0.1" rpy="0 0 0" />
     <axis xyz="0 1 0" rpy="0 0 0"/>
     <parent link="chassis"/>

File: catkin_ws/src/my_robot/urdf/my_robot_2wheel.xacro (robot description, xacro)
@@ -1,4 +1,4 @@
 <robot name="my_robot" xmlns:xacro="http://www.ros.org/wiki/xacro">
-  <xacro:include filename="$(find my_robot)/urdf/my_robot.gazebo" />
+  <xacro:include filename="$(find my_robot)/urdf/my_robot_Differential.gazebo" />
   <link name="robot_footprint"></link>
   <joint name="robot_footprint_joint" type="fixed">
@@ -21,5 +21,5 @@
       <origin xyz="0 0 0" rpy=" 0 0 0"/>
       <geometry>
-        <box size=".5 .2 .1"/>
+        <box size=".4 .2 .1"/>
       </geometry>
     </collision>
@@ -27,5 +27,5 @@
       <origin xyz="0 0 0" rpy=" 0 0 0"/>
       <geometry>
-        <box size=".5 .2 .1"/>
+        <box size=".4 .2 .1"/>
       </geometry>
     </visual>
@@ -56,5 +56,5 @@
   </link>
   <joint type="continuous" name="left_wheel_hinge">
-    <origin xyz="0.15 0.2 0" rpy="0 0 0"/>
+    <origin xyz="0.0 0.15 0" rpy="0 0 0"/>
     <child link="left_wheel"/>
     <parent link="chassis"/>
@@ -87,41 +87,9 @@
     </visual>
   </link>
-  <!-- Left Rear Dummy wheel-->
-  <joint type="continuous" name="left_rear_wheel_hinge">
-    <origin xyz="-0.15 0.2 0" rpy="0 0 0"/>
-    <child link="left_rear_wheel"/>
-    <parent link="chassis"/>
-    <axis xyz="0 1 0" rpy="0 0 0"/>
-    <limit effort="10000" velocity="1000"/>
-    <dynamics damping="1.0" friction="1.0"/>
-  </joint>
-  <link name="left_rear_wheel">
-    <inertial>
-      <mass value="5.0"/>
-      <origin xyz="0 0 0" rpy=" 0 1.57079633 1.57079633"/>
-      <inertia
-          ixx="0.1" ixy="0" ixz="0"
-          iyy="0.1" iyz="0"
-          izz="0.1"
-      />
-    </inertial>
-    <collision name='left_rear_wheel_collision'>
-      <origin xyz="0 0 0" rpy=" 0 1.57079633 1.57079633"/>
-      <geometry>
-        <cylinder radius="0.1" length="0.05"/>
-      </geometry>
-    </collision>
-    <visual name='left_rear_wheel_visual'>
-      <origin xyz="0 0 0" rpy=" 0 1.57079633 1.57079633"/>
-      <geometry>
-        <cylinder radius="0.1" length="0.05"/>
-      </geometry>
-    </visual>
-  </link>
   <!-- RIGHT WHEEL -->
   <joint name="right_wheel_hinge" type="continuous">
     <parent link="chassis"/>
     <child link="right_wheel"/>
-    <origin xyz="0.15 -0.2 0" rpy="0 0 0"/>
+    <origin xyz="0.0 -0.15 0.0" rpy="0 0 0"/>
     <axis xyz="0 1 0"/>
     <limit effort="10000" velocity="1000"/>
@@ -145,36 +113,4 @@
     </collision>
     <visual name="right_wheel_visual">
-      <origin xyz="0 0 0" rpy="0 1.57079633 1.57079633"/>
-      <geometry>
-        <cylinder radius="0.1" length="0.05"/>
-      </geometry>
-    </visual>
-  </link>
-   <!-- Rear Dummy RIGHT WHEEL -->
-  <joint name="right_rear_wheel_hinge" type="continuous">
-    <parent link="chassis"/>
-    <child link="right_rear_wheel"/>
-    <origin xyz="-0.15 -0.2 0" rpy="0 0 0"/>
-    <axis xyz="0 1 0"/>
-    <limit effort="10000" velocity="1000"/>
-    <dynamics damping="1.0" friction="1.0"/>
-  </joint>
-  <link name="right_rear_wheel">
-    <inertial>
-      <mass value="5.0"/>
-      <origin xyz="0 0 0" rpy="0 1.57079633 1.57079633"/>
-      <inertia
-          ixx="0.1" ixy="0" ixz="0"
-          iyy="0.1" iyz="0"
-          izz="0.1"
-      />
-    </inertial>
-    <collision name="right_rear_wheel_collision">
-      <origin xyz="0 0 0" rpy="0 1.57079633 1.57079633"/>
-      <geometry>
-        <cylinder radius="0.1" length="0.05"/>
-      </geometry>
-    </collision>
-    <visual name="right_rear_wheel_visual">
       <origin xyz="0 0 0" rpy="0 1.57079633 1.57079633"/>
       <geometry>
@@ -206,5 +142,5 @@
   </link>
   <joint name="camera_joint" type="fixed">
-    <origin xyz="0.25 0 0" rpy="0 0 0" />
+    <origin xyz="0.20 0 0" rpy="0 0 0" />
     <axis xyz="0 1 0" rpy="0 0 0"/>
     <parent link="chassis"/>
@@ -235,5 +171,5 @@
   </link>
   <joint name="hokuyo_joint" type="fixed">
-    <origin xyz="0.2 0 0.1" rpy="0 0 0" />
+    <origin xyz="0.15 0 0.1" rpy="0 0 0" />
     <axis xyz="0 1 0" rpy="0 0 0"/>
     <parent link="chassis"/>

Commit message: house dervice robot intial commit

File: catkin_ws/src/my_robot/urdf/my_robot.xacro (robot description, xacro)
@@ -3,5 +3,5 @@
   <link name="robot_footprint"></link>
   <joint name="robot_footprint_joint" type="fixed">
-    <origin xyz="0 0 0" rpy="0 0 0" />
+    <origin xyz="0 0 0.05" rpy="0 0 0" />
     <parent link="robot_footprint"/>
     <child link="chassis" />
@@ -21,5 +21,5 @@
       <origin xyz="0 0 0" rpy=" 0 0 0"/>
       <geometry>
-        <box size=".5 .2 .1"/>
+        <box size=".4 .2 .1"/>
       </geometry>
     </collision>
@@ -27,5 +27,5 @@
       <origin xyz="0 0 0" rpy=" 0 0 0"/>
       <geometry>
-        <box size=".5 .2 .1"/>
+        <box size=".4 .2 .1"/>
       </geometry>
     </visual>
@@ -56,5 +56,5 @@
   </link>
   <joint type="continuous" name="left_wheel_hinge">
-    <origin xyz="0.15 0.2 0" rpy="0 0 0"/>
+    <origin xyz="0.0 0.15 0" rpy="0 0 0"/>
     <child link="left_wheel"/>
     <parent link="chassis"/>
@@ -87,17 +87,17 @@
     </visual>
   </link>
-  <!-- Left Rear Dummy wheel-->
-  <joint type="continuous" name="left_rear_wheel_hinge">
-    <origin xyz="-0.15 0.2 0" rpy="0 0 0"/>
-    <child link="left_rear_wheel"/>
-    <parent link="chassis"/>
-    <axis xyz="0 1 0" rpy="0 0 0"/>
+  <!-- RIGHT WHEEL -->
+  <joint name="right_wheel_hinge" type="continuous">
+    <parent link="chassis"/>
+    <child link="right_wheel"/>
+    <origin xyz="0.0 -0.15 0.0" rpy="0 0 0"/>
+    <axis xyz="0 1 0"/>
     <limit effort="10000" velocity="1000"/>
     <dynamics damping="1.0" friction="1.0"/>
   </joint>
-  <link name="left_rear_wheel">
+  <link name="right_wheel">
     <inertial>
       <mass value="5.0"/>
-      <origin xyz="0 0 0" rpy=" 0 1.57079633 1.57079633"/>
+      <origin xyz="0 0 0" rpy="0 1.57079633 1.57079633"/>
       <inertia
           ixx="0.1" ixy="0" ixz="0"
@@ -106,36 +106,4 @@
       />
     </inertial>
-    <collision name='left_rear_wheel_collision'>
-      <origin xyz="0 0 0" rpy=" 0 1.57079633 1.57079633"/>
-      <geometry>
-        <cylinder radius="0.1" length="0.05"/>
-      </geometry>
-    </collision>
-    <visual name='left_rear_wheel_visual'>
-      <origin xyz="0 0 0" rpy=" 0 1.57079633 1.57079633"/>
-      <geometry>
-        <cylinder radius="0.1" length="0.05"/>
-      </geometry>
-    </visual>
-  </link>
-  <!-- RIGHT WHEEL -->
-  <joint name="right_wheel_hinge" type="continuous">
-    <parent link="chassis"/>
-    <child link="right_wheel"/>
-    <origin xyz="0.15 -0.2 0" rpy="0 0 0"/>
-    <axis xyz="0 1 0"/>
-    <limit effort="10000" velocity="1000"/>
-    <dynamics damping="1.0" friction="1.0"/>
-  </joint>
-  <link name="right_wheel">
-    <inertial>
-      <mass value="5.0"/>
-      <origin xyz="0 0 0" rpy="0 1.57079633 1.57079633"/>
-      <inertia
-          ixx="0.1" ixy="0" ixz="0"
-          iyy="0.1" iyz="0"
-          izz="0.1"
-      />
-    </inertial>
     <collision name="right_wheel_collision">
       <origin xyz="0 0 0" rpy="0 1.57079633 1.57079633"/>
@@ -145,36 +113,4 @@
     </collision>
     <visual name="right_wheel_visual">
-      <origin xyz="0 0 0" rpy="0 1.57079633 1.57079633"/>
-      <geometry>
-        <cylinder radius="0.1" length="0.05"/>
-      </geometry>
-    </visual>
-  </link>
-   <!-- Rear Dummy RIGHT WHEEL -->
-  <joint name="right_rear_wheel_hinge" type="continuous">
-    <parent link="chassis"/>
-    <child link="right_rear_wheel"/>
-    <origin xyz="-0.15 -0.2 0" rpy="0 0 0"/>
-    <axis xyz="0 1 0"/>
-    <limit effort="10000" velocity="1000"/>
-    <dynamics damping="1.0" friction="1.0"/>
-  </joint>
-  <link name="right_rear_wheel">
-    <inertial>
-      <mass value="5.0"/>
-      <origin xyz="0 0 0" rpy="0 1.57079633 1.57079633"/>
-      <inertia
-          ixx="0.1" ixy="0" ixz="0"
-          iyy="0.1" iyz="0"
-          izz="0.1"
-      />
-    </inertial>
-    <collision name="right_rear_wheel_collision">
-      <origin xyz="0 0 0" rpy="0 1.57079633 1.57079633"/>
-      <geometry>
-        <cylinder radius="0.1" length="0.05"/>
-      </geometry>
-    </collision>
-    <visual name="right_rear_wheel_visual">
       <origin xyz="0 0 0" rpy="0 1.57079633 1.57079633"/>
       <geometry>
@@ -206,5 +142,5 @@
   </link>
   <joint name="camera_joint" type="fixed">
-    <origin xyz="0.25 0 0" rpy="0 0 0" />
+    <origin xyz="0.20 0 0" rpy="0 0 0" />
     <axis xyz="0 1 0" rpy="0 0 0"/>
     <parent link="chassis"/>
@@ -243,5 +179,5 @@
   </link>
   <joint name="hokuyo_joint" type="fixed">
-    <origin xyz="0.2 0 0.1" rpy="0 0 0" />
+    <origin xyz="0.15 0 0.1" rpy="0 0 0" />
     <axis xyz="0 1 0" rpy="0 0 0"/>
     <parent link="chassis"/>
